File: window_sensor/window_sensor.kicad_pcb (KiCad board)
At the start: 0 parts

Commit message: debugging connectors unified to one
Parts:
- added C1: 5.6pF, Capacitor_SMD:C_0805_2012Metric_Pad1.18x1.45mm_HandSolder, F.Cu at (141.0, 68.5)
- added C2: 5.6pF, Capacitor_SMD:C_0805_2012Metric_Pad1.18x1.45mm_HandSolder, F.Cu at (143.0, 71.5)
- added C3: 4.7uF, Capacitor_SMD:C_0805_2012Metric_Pad1.18x1.45mm_HandSolder, F.Cu at (142.0, 65.5)
- added C4: 100nF, Capacitor_SMD:C_0805_2012Metric_Pad1.18x1.45mm_HandSolder, F.Cu at (148.0, 62.5)
- added C5: 100nF, Capacitor_SMD:C_0805_2012Metric_Pad1.18x1.45mm_HandSolder, F.Cu at (143.0, 73.5)
- added J3: Screw_Terminal_01x02, TerminalBlock:TerminalBlock_Xinya_XY308-2.54-2P_1x02_P2.54mm_Horizontal, F.Cu at (151.5, 79.5)
- added J4: Conn_01x02, Connector_PinHeader_2.54mm:PinHeader_1x02_P2.54mm_Vertical, F.Cu at (157.5, 69.5)
- added J6: Conn_ST_STDC14, Connector_PinHeader_1.27mm:PinHeader_2x07_P1.27mm_Vertical_SMD, F.Cu at (144.2, 80.0)
- added JP1: SolderJumper_2_Bridged, Jumper:SolderJumper-2_P1.3mm_Open_TrianglePad1.0x1.5mm, F.Cu at (140.7, 63.0)
- added JP2: SolderJumper_2_Bridged, Jumper:SolderJumper-2_P1.3mm_Open_TrianglePad1.0x1.5mm, F.Cu at (144.2, 63.0)
- added U1: RFM69HW, RF_Module:HOPERF_RFM69HW, F.Cu at (128.4, 70.0)
- added U2: STM32G031K8Tx, Package_QFP:LQFP-32_7x7mm_P0.8mm, F.Cu at (150.3, 68.7)
- added Y1: 32.768KHz, Crystal:Crystal_SMD_3215-2Pin_3.2x1.5mm, F.Cu at (143.5, 68.5)
Other:
- board outline added: 50.5 x 23.5 mm
- copper layers 0 -> 2
