File: window_sensor/window_sensor.kicad_pcb (KiCad board)
At the start: 2 copper layers, 50.5 x 23.5 mm, 13 parts, among them J3 Screw_Terminal_01x02, J4 Conn_01x02, J6 Conn_ST_STDC14, U1 RFM69HW, U2 STM32G031K8Tx, Y1 32.768KHz

Commit message: pcb updated
Parts:
- added C6: 100nF, Capacitor_SMD:C_0805_2012Metric_Pad1.18x1.45mm_HandSolder, F.Cu at (182.3, 76.6)
- added R1: 100k, Resistor_SMD:R_0805_2012Metric_Pad1.20x1.40mm_HandSolder, F.Cu at (179.3, 76.5)
- added R2: 0, Resistor_SMD:R_0805_2012Metric_Pad1.20x1.40mm_HandSolder, F.Cu at (176.3, 76.5)
- moved U1 34.6 mm to (160.8, 57.8), turned to 90 degrees
- moved JP1 28.0 mm to (167.8, 70.2), turned to -90 degrees
- moved JP2 25.9 mm to (167.8, 73.7), turned to 90 degrees
- moved C4 25.2 mm to (168.3, 77.4), turned to -90 degrees
- moved C3 24.1 mm to (165.3, 71.5), turned to 90 degrees
- moved C1 21.4 mm to (162.3, 70.4), turned to 180 degrees
- moved Y1 19.4 mm to (162.3, 72.9), turned to 0 degrees
- moved J4 17.9 mm to (161.3, 86.9), turned to 90 degrees
- moved C2 16.4 mm to (159.3, 72.4), turned to 90 degrees
- moved U2 16.2 mm to (162.2, 79.7), turned to -90 degrees
- moved C5 14.3 mm to (157.3, 72.5), turned to 90 degrees
- moved J6 9.15 mm to (150.8, 73.7), turned to 0 degrees
- moved J3 1.40 mm to (151.3, 80.9), turned to -90 degrees
Connections:
- J3 pad 1: /WINDOW -> Net-(J3-Pin_1)
- J6 pad 3: unconnected-(J6-VCC-Pad3) -> +BATT
- U1 pad 1: unconnected-(U1-RESET-Pad1) -> Net-(U1-RESET)
- U1 pad 10: unconnected-(U1-ANA-Pad10) -> Net-(AE1-A)
- U2 pad 11: /WINDOW -> unconnected-(U2-PA4-Pad11)
- U2 pad 18: unconnected-(U2-PA8-Pad18) -> /RFM_RESET
- U2 pad 7: unconnected-(U2-PA0-Pad7) -> Net-(J3-Pin_1)
Other:
- board size 50.5 x 23.5 mm -> 23.5 x 50.5 mm

Commit message: First PCB
Parts:
- removed J4: Conn_01x02, Connector_PinHeader_2.54mm:PinHeader_1x02_P2.54mm_Vertical
- removed R2: 0, Resistor_SMD:R_0805_2012Metric_Pad1.20x1.40mm_HandSolder
- added AE1: Antenna, RF_Antenna:NiceRF_SW868-TH13_868Mhz, F.Cu at (111.5, 36.5)
- added BT1: Battery, Battery:BatteryHolder_Keystone_2462_2xAA, B.Cu at (133.0, 89.7)
- added JP3: SolderJumper_2_Bridged, Jumper:SolderJumper-2_P1.3mm_Open_TrianglePad1.0x1.5mm, F.Cu at (138.0, 58.0)
- J2: renamed from J6; footprint Connector_PinHeader_1.27mm:PinHeader_2x07_P1.27mm_Vertical_SMD -> Connector_PinHeader_1.27mm:PinHeader_2x07_P1.27mm_Horizontal
- moved C5 61.8 mm to (120.5, 78.0)
- moved R1 56.8 mm to (122.5, 78.0), turned to 90 degrees
- moved JP1 49.8 mm to (118.0, 74.5), turned to -90 degrees
- moved C4 49.8 mm to (118.5, 78.0)
- moved C2 49.3 mm to (116.5, 78.0), turned to -90 degrees
- moved C1 43.6 mm to (118.7, 69.2)
- moved C3 40.6 mm to (118.7, 71.2), turned to 180 degrees
- moved Y1 40.2 mm to (122.2, 70.2), turned to 90 degrees
- moved J1 40.1 mm to (112.0, 88.5), turned to 0 degrees
- moved JP2 39.5 mm to (138.0, 44.3)
- moved U2 36.1 mm to (125.5, 50.5), turned to 180 degrees
- moved C6 36.0 mm to (121.5, 75.0), turned to 180 degrees
- moved U1 33.7 mm to (129.0, 73.5), turned to 0 degrees
- moved J2 24.4 mm to (129.3, 85.2), turned to -90 degrees
- renumbered C3 to C2, C2 to C3, C6 to C5, C5 to C6, J3 to J1, JP2 to JP1, JP1 to JP2, U2 to U1, U1 to U2
Connections:
- U1 pad 18: /RFM_RESET -> unconnected-(U1-PA8-Pad18)
- U1 pad 23: unconnected-(U2-PA12/PA10-Pad23) -> /RFM_RESET
Routing:
- net +BATT: track 0.00 -> 79.0 mm
- net /RFM_SCK: track 0.00 -> 25.8 mm
- net /RFM_MISO: track 0.00 -> 23.6 mm
- net /SWCLK: track 0.00 -> 22.3 mm, vias 0 -> 2
- net /RST: track 0.00 -> 21.4 mm, vias 0 -> 1
- net /RFM_MOSI: track 0.00 -> 21.2 mm
- net /RFM_CS: track 0.00 -> 21.2 mm, vias 0 -> 2
- net /SWDIO: track 0.00 -> 20.5 mm, vias 0 -> 1
- net Net-(J1-Pin_1): track 0.00 -> 20.2 mm, vias 0 -> 1
- net /RFM_IRQ: track 0.00 -> 19.6 mm, vias 0 -> 2
- net /RFM_RESET: track 0.00 -> 15.2 mm
- net GND: track 0.00 -> 13.3 mm, vias 0 -> 17
- net /UART_TX: track 0.00 -> 11.6 mm, vias 0 -> 1
- net Net-(AE1-A): track 0.00 -> 11.5 mm
- net /UART_RX: track 0.00 -> 9.77 mm, vias 0 -> 2
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- added copper zone on B.Cu, net GND
- added copper zone on F.Cu, net GND
Other:
- board size 23.5 x 50.5 mm -> 33.5 x 60 mm
