File: hw/sensor/sensor.kicad_sch (KiCad schematic)
At the start: 17 parts, among them J1 Screw_Terminal_01x02, J2 Conn_ST_STDC14, U1 STM32G031K8Tx, U2 RFM69HW, Y1 32.768KHz

Commit message: sensor redesigned
Parts:
- removed AE1: Antenna, RF_Antenna:NiceRF_SW868-TH13_868Mhz, symbol Device:Antenna
- added C7: 4.7uF, Capacitor_SMD:C_0805_2012Metric_Pad1.18x1.45mm_HandSolder, symbol Device:C
- added C8, C9: 100nF, Capacitor_SMD:C_0805_2012Metric_Pad1.18x1.45mm_HandSolder, symbol Device:C
- added D1, D2: D_Schottky, Diode_SMD:D_SOD-323_HandSoldering, symbol Device:D_Schottky
- added H1, H4: MountingHole, MountingHole:MountingHole_3.2mm_M3, symbol Mechanical:MountingHole
- added J3: Conn_Coaxial, Connector_Coaxial:SMA_Amphenol_901-143_Horizontal, symbol Connector:Conn_Coaxial
- added JP4: SolderJumper_2_Bridged, Jumper:SolderJumper-2_P1.3mm_Open_TrianglePad1.0x1.5mm, symbol Jumper:SolderJumper_2_Open
- J2: footprint Connector_PinHeader_1.27mm:PinHeader_2x07_P1.27mm_Horizontal -> Connector_PinHeader_1.27mm:PinHeader_2x07_P1.27mm_Vertical
Connections:
- net GND: now also C7.2, C8.2, C9.2, J3.2 (Ext)
- net RFM_RESET: now also U1.17 (PB2); no longer U1.23 (PA12/PA10)
- net at U2.10 (ANA): now also J3.1 (In)
- net RFM_3v3: now reaches JP2.1 (A), U2.8 (3.3V)
- net RFM_3v3: now also C7.1, C8.1, C9.1
- net STM_3v3: now reaches JP1.1 (A), U1.4 (VDD)
- net STM_3v3: now also C2.1, C4.1, C5.1, J2.3 (VCC), R1.1
- removed net +BATT: BT1.1 (+), C2.1, C4.1, C5.1, J2.3 (VCC), JP1.2 (B), JP2.2 (B), R1.1
- new net: D1.1 (K), JP1.2 (B)
- new net: D1.2 (A), D2.2 (A), JP4.2 (B)
- new net: BT1.1 (+), JP4.1 (A)
- new net: D2.1 (K), JP2.2 (B)
- no-connect marks 24 -> 25
Other:
- moved on the sheet: BT1, C1, C2, C3, C4, C5, C6, J1, J2, JP3, R1, U1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
