File: hw/panel/leds.kicad_sch (KiCad schematic)
At the start: 48 parts

Commit message: panel
Parts:
- removed D11, D13, D15, D17, D19, D21, D23, D25, D3, D5, D7, D9: WS2812B-2020, LED_SMD:LED_WS2812B-2020_PLCC4_2.0x2.0mm, symbol LED:WS2812B-2020
- renumbered C7 to C12, C8 to C13, C9 to C14, C10 to C15, C11 to C16, C12 to C17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
Connections:
- net +5V renamed +6V

Commit message: extend top to 200mm
Parts:
- renumbered C12 to C100, C13 to C101, C14 to C102, C15 to C103, C16 to C104, C17 to C105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
